File: Documentation/Arduino_backplane.brd (EAGLE design)
At the start: 101.6 x 53.3 mm, 45 parts, among them IC1 4013N, Q1 BF199, Q5 BF199, X1 M25-HD-20, X2 M25-HD-20

Commit message: Include DAC and new headers to steering and brake headers.
Parts:
- removed C1, C2: (no value), rcl:C025-030X050
- removed R1, R2: (no value), rcl:0204/5
- removed X4, X5, X6, X7, X8: (no value), con-subd:M15HP
- added IC2, IC3: MCP4802, ic-package:DIL08
- added SV1: (no value), con-lstb:MA04-2
- added SV3: Steer, con-lstb:MA04-2
Connections:
- net ADC12 renamed A12
- net ADC14 renamed A14
- net ADC8 renamed A8
- net N$4 renamed A13
- net N$5 renamed A15
- removed net ADC1: ADCL.3, X8.13
- removed net D5: C1.1, R1.1, X3.15, X4.15, X5.15, X6.15, X7.15
- removed net N$14: X3.13, X4.13, X5.13, X6.13, X7.13
- removed net N$16: ADCL.2
- removed net N$17: X3.7, X4.7, X5.7, X6.7, X7.7
- removed net N$18: ADCL.6, X8.10
- removed net N$21: ADCH.4, X3.1, X4.1, X5.1, X6.1, X7.1
- removed net N$7: ADCH.3, X3.2, X4.2, X5.2, X6.2, X7.2
- removed net PL1: XIOL.6
- new net A0: X3.7
- new net A1: ADCL.2, SV1.4
- new net A10: ADCH.3, X3.2
- new net A11: ADCH.4, X3.1
- new net A2: ADCL.3
- new net A3: ADCL.4
- new net A4: ADCL.5, SV3.2
- new net A5: ADCL.6, SV3.4
- new net A9: X3.3
- new net N$5: IC2.3, XIOL.2
- net +5V: now also IC2.1
- net D6: now also SV3.8
- net GND: now also IC2.5, IC2.7, IC3.5, IC3.7; no longer X3.12, X4.11, X4.12, X5.11, X5.12, X6.11, X6.12, X7.11, X7.12
- net INT0: no longer X3.10, X4.10, X4.14, X5.10, X5.14, X6.10, X6.14, X7.10, X7.14
- net N$1: no longer X4.4, X5.4, X6.4, X7.4
- net N$10: now also IC3.8; no longer ADCL.4, X8.12
- net N$12: now also X3.10; no longer ADCL.5, X8.11
- net N$13: no longer X4.5, X5.5, X6.5, X7.5
- net N$15: no longer X4.6, X5.6, X6.6, X7.6
- net N$19: no longer X4.8, X5.8, X6.8, X7.8
- net N$2: now also X3.15; no longer R2.2
- net N$23: now also SV3.6
- net N$3: now also IC2.8, X3.12; no longer C2.1, R1.2, R2.1
- net N$6: now also IC2.6, X3.13; no longer X3.9, X4.9, X5.9, X6.9, X7.9
- net N$8: now also SV1.6; no longer X8.15
- net N$9: now also ADCL.8, SV3.7; no longer X3.3, X4.3, X5.3, X6.3, X7.3
- net PB0: now also IC2.2
- net PB1: no longer XIOL.2
- net PB2: now also IC2.4, IC3.4
- net PB3: no longer XIOL.4
- net PL0: now also IC3.2
- net PL4: now also SV3.5
Routing:
- net PB0: track 63.8 -> 0.00 mm, vias 2 -> 0
- net PL1: track 45.9 -> 0.00 mm
- net PB3: track 113.9 -> 112.1 mm
- net PB1: track 89.7 -> 88.4 mm
Other:
- board text removed: "Arduino Mega 2560 Reference Design"
- board text removed: "Arduino may make changes to specifications and product descriptions at any time, without notice. The Customer must not rely on the absence or characteristics of any features or instructions marked "reserved" or "undefined." Arduino reserves these for future definition and shall have no responsibility whatsoever for conflicts or incompatibilities arising from future changes to them. The product in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"
- board text removed: "D.Cuartielles"
- board text removed: "D.Mellis"
- board text removed: "G.Martino"
- board text removed: "M.Banzi"
- board text removed: "Reference Designs ARE PROVIDED "AS IS" AND "WITH ALL FAULTS. Arduino DISCLAIMS ALL OTHER WARRANTIES, EXPRESS OR IMPLIED, REGARDING PRODUCTS, INCLUDING BUT NOT LIMITED TO, ANY IMPLIED WARRANTIES OF MERCHANTABILITY OR FITNESS FOR A PARTICULAR PURPOSE"
- board text removed: "T.Igoe"
