File: Electronics/Arduino_backplane.brd (EAGLE design)
At the start: 100.3 x 80 mm, 36 parts, among them IC1 4013N, IC2 MCP4802, IC3 MCP4802, Q1 BF199, Q5 BF199, X1 M25-HD-20, X2 M25-HD-20

Commit message: Modifications by Tyler and Charles on March 14.
Parts:
- removed IC1: 4013N, 40xx:DIL14
- added IC4: 4013N, ic-package:DIL14
Connections:
- removed net N$2: C4.1, IC1.9, R5.1
- removed net N$25: IC1.11, JP5.6
- removed net N$27: JP7.2, R7.2
- removed net N$30: IC1.3, JP5.8, JP7.3
- removed net N$34: IC1.12, R5.2
- removed net N$35: C3.1, IC1.5, R6.1
- removed net N$36: C5.2, IC1.10, IC1.4, R4.1
- removed net N$38: IC1.2, R6.2
- removed net N$39: Q1.1, R7.1
- removed net N$4: IC1.1, JP7.1
- removed net N$5: IC1.13, R3.2
- removed net VDD: IC1.14
- removed net VSS: IC1.7
- new net CLKA: IC4.3, JP5.8, JP7.3
- new net CLKB: IC4.11, JP5.6
- new net DA: C3.1, IC4.5, R6.1
- new net DB: C4.1, IC4.9, R5.1
- new net N$11: JP7.2, R7.1
- new net N$12: Q1.1, R7.2
- new net QA: IC4.1, JP7.1
- new net QB: R3.2
- new net RA: C5.2, IC4.10, IC4.4, R4.1
- new net ~QA: IC4.2, R6.2
- new net ~QB: IC4.12, R5.2
- net +5V: now also IC4.14
- net GND: now also IC4.6, IC4.7, IC4.8; no longer IC1.6, IC1.8
Routing:
- net 5VBRK: track 177.4 -> 0.00 mm, vias 2 -> 0
- net D48: track 105.5 -> 0.00 mm, vias 2 -> 0
- net CLKB: track 0.00 -> 94.4 mm, vias 0 -> 3
- net VCC: track 102.6 -> 192.9 mm, vias 1 -> 2
- net CLKA: track 0.00 -> 81.2 mm, vias 0 -> 3
- net QA: track 0.00 -> 80.3 mm
- net N$25: track 65.3 -> 0.00 mm, vias 1 -> 0
- net D43: track 104.3 -> 164.3 mm
- net A14: track 58.4 -> 116.7 mm, vias 0 -> 1
- net N$30: track 53.4 -> 0.00 mm, vias 1 -> 0
- net RA: track 0.00 -> 52.5 mm, vias 0 -> 3
- net N$36: track 51.0 -> 0.00 mm, vias 1 -> 0
- net DA: track 0.00 -> 47.1 mm, vias 0 -> 1
- net D19INT3: track 119.7 -> 76.9 mm, vias 3 -> 4
- net A0: track 58.7 -> 100.4 mm, vias 0 -> 2
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