File: Electronics/C1_Interface.sch (EAGLE design)
At the start: 44 parts, among them J1 PIN1-2, J2 PIN1-2, J3 PIN1-2

Commit message: 3 new boards
Parts:
- removed J1: PIN1-2, con-faston:PIN1-2
- removed LED_1, LED_2, LED_3, LED_4, LED_5, LED_6, LED_7, LED_8: (no value), led:LEDB156
- removed LED_10: Cruise LED, led:LEDB156
- removed LED_11: On LED, led:LEDB156
- removed LED_12: Motor LED, led:LEDB156
- removed LED_13: Brake LED, led:LEDB156
- removed LED_14: Steer LED, led:LEDB156
- removed LED_15: Reverse LED, led:LEDB156
- removed LED_9: Stop LED, led:LEDB156
- removed R11, R14, R15, R18, R19, R20, R22, R24, R25, R26, R5: 1K, resistor:R-US_0204/7
- removed R2, R3: 200, resistor:R-US_0204/7
- removed R27, R28, R4: 220, resistor:R-US_0204/7
- removed R29: 10K, resistor:R-US_0204/7
- removed S1: Motor, switch:M9040P
- removed S2: Brake, switch:M9040P
- removed S3: Steer, switch:M9040P
- removed S4: On, switch:M9040P
- removed S5: Cruise Switch, switch-misc:DTE6K
- removed S6: Stop switch, switch-misc:DTE6K
- removed S7: Reverse Switch, switch-misc:DTE6K
- added D1: 1N4004, diode:1N4004
- added IC1: ACS750LCA-050, allegro:ACS750LCA-050
- added J10: PIN1-2, con-faston:PIN1-2
- added K2: JW1A, relay:JW1A
- added LED1: (no value), led:LED3MM
- added X2, X4: SSW-103-02-S-D, con-samtec:SSW-103-02-S-D
- added X3: SSW-102-02-S-Q, con-samtec:SSW-102-02-S-Q
- R1: value 200 -> 10K; device resistor:R-US_0204/7 -> rcl:R-US_0204/5
- X1: device con-subd:M25-182 -> con-subd:F15H
Connections:
- removed net N$16: LED_1.C, R11.2
- removed net N$19: R27.2, X1.17
- removed net N$21: LED_12.A, R2.2
- removed net N$22: LED_15.A, X1.11
- removed net N$23: LED_12.C, S1.P
- removed net N$24: LED_13.C, S2.P
- removed net N$25: LED_9.C, R25.1
- removed net N$26: LED_9.A, X1.10
- removed net N$27: LED_14.A, R3.2
- removed net N$28: R2.1, X1.8
- removed net N$29: LED_13.A, R1.2
- removed net N$30: LED_14.C, S3.P
- removed net N$31: R4.2, X1.12
- removed net N$32: R1.1, X1.7
- removed net N$33: R4.1, S7.P, S7.P@1
- removed net N$34: R27.1, S5.P, S5.P@1
- removed net N$35: R28.2, X1.18
- removed net N$37: R28.1, S6.P, S6.P@1
- removed net N$38: LED_2.C, R5.2
- removed net N$39: X1.19
- removed net REVERSE: LED_15.C, R26.1
- net +5V: now also IC1.VCC, X1.14, X2-3.1, X3-1.1; no longer J3.1, S1.S, S2.S, S3.S, S4.S, S5.S, S5.S@1, S6.S, S6.S@1, S7.S, S7.S@1, X1.24
- net GND: now also IC1.GND, X1.11, X2-5.1, X3-3.1, X4-5.1; no longer J1.1, R11.1, R14.1, R15.1, R18.1, R19.1, R20.1, R22.1, R24.2, R25.2, R26.2, R29.2, R5.1, S1.O, S2.O, S3.O, S4.O, X1.25
- net N$1: now also D1.C, J10.1, K2_.1, LED1.A; no longer R3.1, X1.6
- net N$10: now also D1.A, K2_.2, R1.1, X1.6; no longer LED_5.C, R18.2
- net N$11: now also X1.1, X2-2.1; no longer LED_5.A, X1.2
- net N$12: now also IC1.IP-, J2.1; no longer LED_6.C, R19.2
- net N$13: now also X1.2, X2-4.1; no longer LED_6.A, X1.1
- net N$14: now also X1.3, X2-6.1; no longer LED_7.C, R20.2
- net N$15: now also X2-1.1; no longer LED_10.A
- net N$17: now also X1.12, X3-2.1; no longer J2.1, LED_11.A, S4.P
- net N$18: now also X1.15, X4-6.1; no longer LED_11.C, R29.1
- net N$2: now also X1.4, X4-1.1; no longer LED_8.C, R22.2
- net N$20: now also IC1.IP+, K21.P; no longer LED_7.A, X1.15
- net N$3: now also IC1.VOUT, X1.7; no longer LED_10.C, R24.1
- net N$4: now also LED1.C, R1.2; no longer LED_3.C, R14.2
- net N$5: now also X1.8, X3-4.1; no longer LED_3.A, X1.4
- net N$6: now also J3.1, K21.S; no longer LED_4.C, R15.2
- net N$7: now also X1.10, X4-2.1; no longer LED_4.A, X1.3
- net N$8: now also X4-3.1; no longer LED_1.A
- net N$9: now also X1.13, X4-4.1; no longer LED_8.A, X1.16
Other:
- note added: "Analog B"
- note added: "Analog throttle"
- note added: "D43"
- note added: "D48"
- note added: "Fuel (36 V signal)"
- note added: "Joystick Center"
- note added: "Motion joystick"
- note added: "Motor current"
- note added: "Normally open"
- note added: "Orange Anderson 12V"
- note added: "PWM throttle"
- note added: "Red Anderson 36V"
- note added: "Reverse Cmd out"
- note added: "Steer joystick"
- note added: "Wireless E-stop"
- note added: "~Estop"
- note removed: "36V fuel"
- note removed: "5V"
- note removed: "Black Anderson"
- note removed: "Cruise Button"
- note removed: "Cruise LED"
- note removed: "Enable Brake"
- note removed: "Enable Steer"
- note removed: "Enable Throttle"
- note removed: "GND"
- note removed: "LED 1"
- note removed: "LED 3"
- note removed: "LED 4"
- note removed: "LED 5"
- note removed: "LED 6"
- note removed: "LED 7"
- note removed: "LED 8"
- note removed: "Orange Anderson"
- note removed: "Reverse button"
- note removed: "Stop Button"
- note removed: "Stop LED"
- note removed: "To C2 Box"
- moved on the sheet: J2, J3, R1
