File: Electronics/MegaShieldTrio.brd (EAGLE design)
At the start: 99.8 x 80 mm, 56 parts, among them X1 Vehicle control, X2 2odo__, X3 1odo__, X4 RJ45-8L-B, X5 RJ45-8L-B

Commit message: Moved ICSP
Parts:
- moved ICSP 5.08 mm to (48.3, 61.0)
- moved C6D78-85 1.27 mm to (87.6, 6.35)
- moved C6D8-13 1.27 mm to (87.6, 2.54)
Routing:
- net NAV_FIX: track 133.8 -> 189.8 mm, vias 6 -> 9
- net LED1: track 189.7 -> 146.5 mm, vias 10 -> 15
- net 4D5_6A14: track 89.1 -> 102.6 mm, vias 4 -> 5
- net INU_BRN: track 139.7 -> 149.1 mm, vias 7 -> 11
- net R2RNG: track 197.3 -> 189.0 mm, vias 8 -> 9
- net MISO: track 191.2 -> 184.5 mm
- net FL_RNG: track 174.3 -> 167.8 mm
- net L_RNG: track 144.0 -> 149.4 mm, vias 9 -> 11
- net +5V: track 364.1 -> 367.5 mm
- net 4D6_6A15: track 122.8 -> 125.2 mm, vias 11 -> 9
- net F_RNG: track 138.2 -> 139.8 mm
- net CHN1: track 172.4 -> 170.8 mm
- net MOSI: track 189.3 -> 187.9 mm
- net VIN: track 172.4 -> 171.5 mm
- net C6AVL: track 167.3 -> 166.5 mm, vias 4 -> 6
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