File: Electronics/MegaShieldTrioV2.sch (EAGLE design)
At the start: 37 parts, among them X1 Vehicle control, X2 2odo__, X3 1odo__, X4 RJ45-8L-B, X5 S5B-ZR, X6 S6B-ZR, X7 22-23-2031

Commit message: Added four new boards to Electronics
Parts:
- removed C2, C3: 1 uF, rcl:C-US025-030X050
- removed C4L, C4R: (no value), pinhead:PINHD-1X17
- removed IC1: (no value), ic-package:DIL8
- removed INU: CHR_UM6, Elcano:CHR_UM6
- removed JP_C3: (no value), pinhead:PINHD-1X6
- removed JP_C5_C4, SHIELD_A0-5, SHIELD_PWR: (no value), pinhead:PINHD-2X6
- removed MOUSE: Visual odometry, pinhead:PINHD-1X10
- removed R2: 4.7 K, rcl:R-US_0207/10
- removed SHIELD_D0-7, SHIELD_D8-13: (no value), pinhead:PINHD-2X8
- removed X5: S5B-ZR, con-jst1:S4B-ZR
- removed X6: S6B-ZR, con-jst:S4B-ZR
- removed X7: 22-23-2031, con-molex:22-23-2031
- added C6: 0.1uF, capacitor-wima:C2.5/2
- added DAC: MCP 4802, ic-package:DIL8
- added IC3: DS 8291, ic-package:DIL8
- added JP3: Turns, pinhead:PINHD-1X6
- added LSM303: (no value), pinhead:PINHD-1X8
- added R4: 100, resistor:R-US_0204/5
- C3L: value (none) -> Pilot digital
- C3R: value (none) -> Pilot analog
- C6D14-21: value C6 Digital 14-21 -> GPS; device Elcano:PINHD-1X8SMALL8 -> pinhead:PINHD-1X8
- D22-53: value (none) -> High digital
- IC2: value (none) -> DS 8291
- X1: value Vehicle control -> RJ45-8L-B; device con-subd:M25H -> con-tycoelectronics:RJ45-8L-B
- X2: value 2odo__ -> Vehicle control; device Elcano:ODO_JACK -> con-subd:M25H
- X3: value 1odo__ -> 2odo__
- renumbered JP2 to D22-53
Connections:
- removed net 3.3V: C3R.16, MOUSE.3, POWER.5, SHIELD_PWR.3
- removed net 4D5_6A14: C4L.10, C6A8-15.2, SHIELD_D0-7.6
- removed net 4D6_6A15: C4L.11, C6A8-15.1, SHIELD_D0-7.4
- removed net 4D7_6D43: C4L.12, SHIELD_D0-7.2
- removed net 6D10_2A6: X1.23
- removed net AREF: C3R.15, C4R.15, C6D8-13.1, SHIELD_D8-13.1, SHIELD_D8-13.2
- removed net C2STAT: C6D14-21.4, X1.19
- removed net C4AVL: C3L.7, C4L.8, SHIELD_D0-7.10, SHIELD_D0-7.11
- removed net C4D12: C4L.17, C4R.2, SHIELD_D8-13.8
- removed net C6AVL: C4L.7, SHIELD_D0-7.12
- removed net C6D10: C6D8-13.6
- removed net CLICK1: C3.2, C6D0-7.6, R2.1, X1.21, X3.1
- removed net CLICK2: C4.2, C6D0-7.5, R1.1, X2.1
- removed net CRS_BRK: C3L.10, C6A0-7.6, SHIELD_D0-7.5, X1.7
- removed net CRS_STR: C6A0-7.7, X1.6
- removed net CRS_THR: C6A0-7.8, X1.8
- removed net D39: D22-53.20
- removed net D41: D22-53.22
- removed net DACA: IC1.8, X7-1.S
- removed net DACB: IC1.6, X7-3.S
- removed net DRV_CMD: X1.18
- removed net F2RNG: C4R.12, SHIELD_A0-5.12
- removed net FL_RNG: C4R.8, SHIELD_A0-5.4
- removed net GPS_CNTRL: C6D14-21.1, INU.10, X6-1.1
- removed net GPS_LOC: C6D14-21.2
- removed net GPS_PPS: C6D14-21.7
- removed net GPS_PWR: C6D8-13.7
- removed net INU_BRN: C6D14-21.6
- removed net INU_CNTRL: C6D14-21.5
- removed net INU_SS: INU.5
- removed net LED4: X1.3
- removed net L_RNG: C3R.10, C4R.10, SHIELD_A0-5.7, SHIELD_A0-5.8
- removed net MISO: C6D8-13.4, D22-53.31, IC1.2, ICSP.1, INU.7, MOUSE.5, X6-4.1
- removed net MOSI: C6D8-13.5, D22-53.32, IC1.4, ICSP.4, INU.8, MOUSE.6, X6-3.1
- removed net MOUSE_SS: D22-53.34, MOUSE.4
- removed net MOV_OK: C4L.9, C6D0-7.4, SHIELD_D0-7.8, X1.17
- removed net N$1: INU.4, X5-2.1
- removed net N$11: C2.1, X3.2, X3.3
- removed net N$17: INU.12, X5-5.1
- removed net N$2: INU.9, X6-2.1
- removed net N$24: POWER.1
- removed net N$27: C4R.6, SHIELD_PWR.6
- removed net N$3: INU.13, X5-4.1
- removed net N$36: C3R.17, SHIELD_D8-13.5
- removed net N$38: C3L.3, SHIELD_D0-7.13
- removed net N$39: ICSP.2, INU.1, X5-3.1
- removed net N$4: C3R.7, SHIELD_A0-5.1
- removed net N$40: C3R.6, SHIELD_PWR.5
- removed net N$41: C3L.8, SHIELD_D0-7.9
- removed net N$42: C3R.8, SHIELD_A0-5.3
- removed net N$45: C3R.11, SHIELD_A0-5.9
- removed net N$46: C3R.12, SHIELD_A0-5.11
- removed net N$47: C3R.1, C3R.14, JP_C3.2
- removed net N$48: C4R.1, C4R.14
- removed net N$49: C4R.11, SHIELD_A0-5.10
- removed net N$5: C4R.7, SHIELD_A0-5.2
- removed net N$51: C4R.17, SHIELD_D8-13.6
- removed net N$53: C3L.9, SHIELD_D0-7.7
- removed net N$54: C3L.11, SHIELD_D0-7.3
- removed net N$55: C3L.12, SHIELD_D0-7.1
- removed net N$57: C3L.14, SHIELD_D8-13.13
- removed net N$59: C3L.17, JP_C3.3, SHIELD_D8-13.7
- removed net N$6: X6-6.1
- removed net N$60: C3L.2, C3R.13, JP_C3.1
- removed net N$8: C4R.16, SHIELD_PWR.4
- removed net NAV_FIX: C4L.4, C6D14-21.3, SHIELD_D0-7.16
- removed net NPD: D22-53.28, MOUSE.9
- removed net PATH: C4L.3, SHIELD_D0-7.14, SHIELD_D0-7.15
- removed net SCK: ICSP.3, INU.6, MOUSE.7, X6-5.1
- removed net SCLK: D22-53.33, IC1.3
- removed net SNR_SEL: C4L.2, C4R.13, JP_C5_C4.2
- removed net SNR_SO: C4L.1, C4L.16, SHIELD_D8-13.10
- removed net SPD_LMT: C4L.14, C6A8-15.8, SHIELD_D8-13.14, X1.9
- removed net SPEED: C3L.1, C3L.16, C6A8-15.3, SHIELD_D8-13.9, X1.10
- removed net SS2_3: C3L.13, JP_C3.5, SHIELD_D8-13.15
- removed net SS2_3/4: C6D0-7.7, JP_C5_C4.9, X1.22
- removed net SS2_4: C4L.13, JP_C5_C4.10, SHIELD_D8-13.16
- removed net SS3/4_6: C6A8-15.4, JP_C5_C4.11
- removed net SS3_6: C3L.15, JP_C3.6, SHIELD_D8-13.11
- removed net SS4_2: C6D0-7.8, X1.20
- removed net SS4_6: C4L.15, JP_C5_C4.12, SHIELD_D8-13.12
- removed net S_SCK: JP_C5_C4.3, X4.6
- removed net S_SI: IC2.2, JP_C5_C4.5
- removed net S_SO: IC2.3, JP_C5_C4.7
- removed net S_SS: JP_C5_C4.1, X4.3
- new net 2TX6RX: C6D14-21.4, X2.19
- new net 3MISO: C3L.17, C3R.2, IC2.3, IC3.3
- new net 3MOSI: C3L.1, C3L.16, DAC.4, IC2.2, IC3.2
- new net 3SCK: C3R.1, C3R.17, C3R.7, DAC.3, X1.3, X4.3
- new net 3SS5F: C3L.15, C3L.2, C3R.8, X1.6
- new net 3SS5R: C3L.13, X4.6
- new net 3SS_DAC: C3L.14, DAC.2
- new net 3TX2RX: C3L.3, X2.18
- new net 3V3: LSM303.1, LSM303.2, POWER.5
- new net 5V_C3: C3R.6, DAC.1
- new net 6MISO: C6D8-13.4, D22-53.31, ICSP.1
- new net 6MOSI: C6D8-13.5, D22-53.32, ICSP.4
- new net 6SCK: C6D8-13.3, D22-53.33, ICSP.3
- new net 6SCL: C6D14-21.8, LSM303.8
- new net 6SDA: C6D14-21.7, LSM303.7
- new net 6TX2RX: C6D14-21.5, X2.20
- new net A0: C3R.14, C6A0-7.1
- new net A1: C3R.13, C6A0-7.2
- new net A5: C3R.9, C6A0-7.6
- new net ACK26: C6D0-7.4, X2.17
- new net ACK34: C3R.11, X2.9
- new net ACK43: C3L.10, C3R.10, C6A0-7.5
- new net ACK62: C6D0-7.3, X2.22
- new net AUTREQ: C3L.9, C6D0-7.5, X2.7
- new net CLICK: C4.2, C6D0-7.6, R1.1, X2.21, X3.1
- new net CRSSTR: DAC.6, X2.6
- new net CRSTHR: DAC.8, X2.8
- new net D09: D22-53.18, X2.14
- new net DRDY: D22-53.11, LSM303.4
- new net I1LSM: C6D14-21.6, LSM303.6
- new net I2LSM: D22-53.9, LSM303.5
- new net MANRQ: C3L.11, X2.10
- new net MISO+R: IC3.6, X4.5
- new net MISO-R: IC3.5, X4.4
- new net MOSI+R: IC3.8, R4.1, X4.8
- new net MOSI-R: IC3.7, R4.2, X4.7
- new net RDY26: D22-53.16, X2.12
- new net RDY32: C3L.12, X2.11
- new net RDY62: C6D0-7.2, X2.23
- new net STR_L: C6A0-7.3, JP3.3
- new net STR_R: C6A0-7.4, JP3.4
- net +5V: now also C6.1, IC3.1, ICSP.2, JP3.1, JP3.6, POWER.7, X2.24; no longer C3.1, D22-53.1, D22-53.2, IC1.1, MOUSE.2, R2.2, X1.24
- net CRS_RVS: now also C3L.8, X2.13; no longer X1.13
- net GND: now also C6.2, DAC.5, DAC.7, IC3.4, JP3.2, JP3.5, LSM303.3, X1.1, X2.25, X4.1; no longer C2.2, C4L.6, C4R.4, C6D8-13.2, D22-53.35, D22-53.36, IC1.5, IC1.7, INU.2, INU.3, MOUSE.1, SHIELD_D8-13.3, SHIELD_D8-13.4, SHIELD_PWR.10, SHIELD_PWR.7, SHIELD_PWR.8, SHIELD_PWR.9, X1.25, X4.8, X5-1.1, X7-2.S
- net LED1: now also X2.5; no longer X1.5
- net LED3: now also C3R.12, X2.4; no longer X1.4
- net LED5: now also X2.2; no longer MOUSE.10, X1.2
- net LED6: now also D22-53.17, X2.1; no longer X1.1
- net LED7: now also D22-53.14, X2.15; no longer X1.15
- net LED8: now also D22-53.12, X2.16; no longer C6D14-21.8, X1.16
- net MISO+: now also X1.5; no longer X4.4
- net MISO-: now also X1.4; no longer X4.5
- net MOSI+: now also X1.8; no longer X4.1
- net MOSI-: now also X1.7; no longer X4.2
- net N$23: now also X3.2, X3.3; no longer X2.2, X2.3
- net RESET: no longer C4L.5, C4R.5, MOUSE.8, SHIELD_PWR.1, SHIELD_PWR.2
- net VIN: now also POWER.1, X1.2, X4.2; no longer C3R.9, C4R.3, C4R.9, SHIELD_A0-5.5, SHIELD_A0-5.6, SHIELD_PWR.11, SHIELD_PWR.12, X4.7
Other:
- note added: "A8"
- note added: "AREF"
- note added: "C3_SS"
- note added: "D25"
- note added: "D27"
- note added: "D28"
- note added: "D29"
- note added: "D31"
- note added: "D33"
- note added: "D34"
- note added: "D35"
- note added: "D41"
- note added: "D45"
- note added: "D47"
- note added: "D53"
- note added: "DRDY"
- note added: "GPS"
- note added: "I1"
- note added: "I2"
- note added: "Vision"
- note removed: "3V"
- note removed: "ARef"
- note removed: "Bearing"
- note removed: "C4 Data Available"
- note removed: "C4 MISO"
- note removed: "C4 MOSI"
- note removed: "C6 Data Available"
- note removed: "CH Robotics UM6"
- note removed: "D1 (Tx2)"
- note removed: "D2 (Rx2)"
- note removed: "D3 (MOSI)"
- note removed: "D39"
- note removed: "D4 (MISO)"
- note removed: "D5 (SCK)"
- note removed: "D6 (SS)"
- note removed: "GPS Location"
- note removed: "GPS control"
- note removed: "INU Control"
- note removed: "LED"
- note removed: "NCS"
- note removed: "NPD"
- note removed: "Optical Mouse"
- note removed: "Pgm"
- note removed: "Rx"
- note removed: "SNR_SCK"
- note removed: "SNR_SI"
- note removed: "SNR_SO"
- note removed: "SNR_SS"
- note removed: "Spare"
- note removed: "Speed Limit"
- note removed: "Tilt SS"
- note removed: "Tx"
- note removed: "UM7"
- note removed: "Vin"
- moved on the sheet: C1, C3R, C4, C5, C6A0-7, IC2, ICSP, R1, R3, X3, X4
